File: sfp-plus-mod.kicad_pcb (KiCad board)
At the start: 4 copper layers, 110.3 x 22 mm, 6 parts, among them J1 sfp-plus-mod, J11 Conn_Coaxial, J12 Conn_Coaxial, J2 PMOD 2x6, J21 Conn_Coaxial, J22 Conn_Coaxial

Commit message: sfp-plus-mod-1.1
Parts:
- added svg2mod: G***, library:lsi-logo-16mm, F.Cu at (200.2, 110.0)
Other:
- board text added: "sfp-plus-mod-1.1"

Commit message: sfp-plus-mod-1.2
Other:
- board text added: "sfp-plus-mod-1.2"
- board text removed: "sfp-plus-mod-1.1"
Changed lines of the file:
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@@
         (effects (font (size 0.2 0.2) (thickness 0.05)) (justify left bottom))
     )
+    (fp_poly
+      (pts
+        (xy -2.2 -4.6)
+        (xy -2.2 4.6)
+        (xy 1.3 4.6)
+        (xy 1.3 -4.6)
+      )
+      (stroke (width 0.1) (type solid)) (fill solid) (layer "B.Mask"))
+    (fp_poly
+      (pts
+        (xy -2.2 -4.6)
+        (xy -2.2 4.6)
+        (xy 1.3 4.6)
+        (xy 1.3 -4.6)
+      )
+      (stroke (width 0.1) (type solid)) (fill solid) (layer "F.Mask"))
     (fp_line (start 1.7 0) (end 2.3 -1)
       (stroke (width 0.12) (type solid)) (layer "Dwgs.User"))
@@
     (effects (font (size 1.5 1.5) (thickness 0.3) bold) (justify left bottom))
   )
-  (gr_text "sfp-plus-mod-1.1" (at 191.7 90.8) (layer "F.SilkS")
+  (gr_text "sfp-plus-mod-1.2" (at 191.7 90.8) (layer "F.SilkS")
     (effects (font (size 1 1) (thickness 0.2) bold) (justify left bottom))
   )

Commit message: sfp-plus-mod-1.3
Parts:
- added ?: , library:mount_hole, F.Cu at (167.0, 94.0)
- added ?: , library:mount_hole, F.Cu at (197.0, 94.0)
- added ?: , library:mount_hole, F.Cu at (197.0, 106.0)
- added ?: , library:mount_hole, F.Cu at (167.0, 106.0)
- moved svg2mod 12.5 mm to (192.0, 100.5)
Other:
- board text added: "sfp-plus-mod-1.3"
- board text removed: "sfp-plus-mod-1.2"
