File: sfp-plus-mod.kicad_pcb (KiCad board)
At the start: 4 copper layers, 110.3 x 22 mm, 11 parts, among them J1 sfp-plus-mod, J11 Conn_Coaxial, J12 Conn_Coaxial, J2 PMOD 2x6, J21 Conn_Coaxial, J22 Conn_Coaxial

Commit message: sfp-plus-mod-1.3-5
Routing:
- net GND: track 9.60 -> 14.7 mm
Other:
- board text added: "sfp-plus-mod-1.3-5"
- board text removed: "sfp-plus-mod-1.3"
Changed lines of the file:
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@@
 		)
 	)
-	(gr_text "sfp-plus-mod-1.3"
+	(gr_text "sfp-plus-mod-1.3-5"
 		(at 191.7 90.8 0)
 		(layer "F.SilkS")
@@
 	)
 	(segment
+		(start 102.65 103.4)
+		(end 100.7 103.4)
+		(width 0.2)
+		(layer "B.Cu")
+		(net 4)
+	)
+	(segment
+		(start 103.05 96.6)
+		(end 102.65 96.2)
+		(width 0.2)
+		(layer "B.Cu")
+		(net 4)
+	)
+	(segment
+		(start 103.1 103.8)
+		(end 103.05 103.8)
+		(width 0.2)
+		(layer "B.Cu")
+		(net 4)
+	)
+	(segment
+		(start 102.65 96.2)
+		(end 100.7 96.2)
+		(width 0.2)
+		(layer "B.Cu")
+		(net 4)
+	)
+	(segment
+		(start 103.05 103.8)
+		(end 102.65 103.4)
+		(width 0.2)
+		(layer "B.Cu")
+		(net 4)
+	)
+	(segment
 		(start 102.925001 102.825)
 		(end 161.4932 102.825)
@@
 		(min_thickness 0.25)
 		(filled_areas_thickness no)
-		(fill yes
+		(fill
 			(thermal_gap 0.5)
 			(thermal_bridge_width 0.5)
@@
 		(min_thickness 0.25)
 		(filled_areas_thickness no)
-		(fill yes
+		(fill
 			(thermal_gap 0.5)
 			(thermal_bridge_width 0.5)

Commit message: sfp-plus-mod-1.4
Connections:
- J1 pad 1: GND -> VeeT
- J1 pad 10: GND -> VeeR
- J1 pad 11: GND -> VeeR
- J1 pad 14: GND -> VeeR
- J1 pad 15: VCC -> VccR
- J1 pad 16: VCC -> VccT
- J1 pad 17: GND -> VeeT
- J1 pad 20: GND -> VeeT
- J11 pad 2: GND -> VeeR
- J12 pad 2: GND -> VeeR
- J2 pad 11: GND -> VeeT
- J2 pad 12: VCC -> VccT
- J2 pad 5: GND -> VeeR
- J2 pad 6: VCC -> VccR
- J21 pad 2: GND -> VeeT
- J22 pad 2: GND -> VeeT
Routing:
- net VeeT: track 0.00 -> 27.5 mm, vias 0 -> 2
- net VccT: track 0.00 -> 23.5 mm, vias 0 -> 1
- net VeeR: track 0.00 -> 23.2 mm, vias 0 -> 2
- net VccR: track 0.00 -> 19.4 mm, vias 0 -> 1
- net GND: track 14.7 -> 0.00 mm, vias 4 -> 0
- net VCC: track 6.93 -> 0.00 mm, vias 2 -> 0
- added copper zone on In2.Cu, net VccR
- added copper zone on In2.Cu, net VccT
- added copper zone on In1.Cu, net VeeR
- added copper zone on In1.Cu, net VeeT
- removed copper zone on In1.Cu, net GND
- removed copper zone on In2.Cu, net VCC
Other:
- board text added: "sfp-plus-mod-1.4"
- board text removed: "sfp-plus-mod-1.3-5"
