File: sfp-plus-mod.kicad_sch (KiCad schematic)
At the start: 6 parts, among them J1 sfp-plus-mod, J11 Conn_Coaxial, J12 Conn_Coaxial, J2 PMOD 2x6, J21 Conn_Coaxial, J22 Conn_Coaxial

Commit message: sfp-plus-mod-1.4
Connections:
- net GND renamed VeeR
- net VeeR: no longer J1.1 (VeeT), J1.17 (VeeT), J1.20 (VeeT), J2.11 (Pin_11), J21.2 (Ext), J22.2 (Ext)
- net VCC renamed VccR
- net VccR: no longer J1.16 (VccT), J2.12 (Pin_12)
- new net VccT: J1.16 (VccT), J2.12 (Pin_12)
- new net VeeT: J1.1 (VeeT), J1.17 (VeeT), J1.20 (VeeT), J2.11 (Pin_11), J21.2 (Ext), J22.2 (Ext)
