File: addons/addon-eeprom.kicad_sch (KiCad schematic)
At the start: 6 parts, among them J1 sfp-plus-mod, J11 Conn_Coaxial, J12 Conn_Coaxial, J2 PMOD 2x6, J21 Conn_Coaxial, J22 Conn_Coaxial

Commit message: sfp-plus-mod-1.3-4
Parts:
- removed J1: sfp-plus-mod, library:sfp-plus-mod, symbol sfp-plus-mod:sfp-plus-mod
- removed J11, J12, J21: Conn_Coaxial, Connector_Coaxial:SMA_Wurth_60312002114503_Vertical, symbol Connector:Conn_Coaxial
- removed J22: Conn_Coaxial, Connector_Coaxial:SMA_Amphenol_901-144_Vertical, symbol Connector:Conn_Coaxial
- added R1, R2, R4: 0, Resistor_SMD:R_0402_1005Metric, symbol Device:R
- added U1: AT24CS02-XHM, Package_SO:TSSOP-8_4.4x3mm_P0.65mm, symbol Memory_EEPROM:AT24CS02-XHM
Connections:
- net GND: now also R1.1, R2.1, R4.1, U1.1 (A0), U1.2 (A1), U1.3 (A2), U1.4 (GND), U1.7 (WP)
- net MOD_ABS: now also R2.2
- net RX_LOS: now also R1.2
- net SCL: now also U1.6 (SCL)
- net SDA: now also U1.5 (SDA)
- net TX_FAULT: now also R4.2
- net VCC: now also U1.8 (VCC)
